File: axis_pcb_v3/axis_pcb_v3.kicad_pcb (KiCad board)
At the start: 2 copper layers, 140.5 x 91 mm, 31 parts, among them J1 7.2V, J10 ICM0948, J11 TB6612FNG_RIGHT, J12 EncoderA, J13 MotorA, J14 MotorB, J15 EncoderB, J16 Power_Switch, J2 LM2596-IN+, J3 LM2596-IN-, J4 LM2596-OUT+, J5 LM2596-OUT-, J6 ESP-32-LEFT, J7 LCD-2x16, J8 ESP-32-RIGHT, J9 TB6612FNG_LEFT

Commit message: Add files via upload
Routing:
- net GND: track 0.00 -> 9.27 mm, vias 0 -> 4
Changed lines of the file:
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@@
 		(tenting front back)
 		(pcbplotparams
-			(layerselection 0x00000000_00000000_55555555_5755f5ff)
-			(plot_on_all_layers_selection 0x00000000_00000000_00000000_00000000)
+			(layerselection 0x00000000_00000000_5555555f_5755f5ff)
+			(plot_on_all_layers_selection 0x00000000_00000000_00000000_02000000)
 			(disableapertmacros no)
 			(usegerberextensions no)
@@
 			(plotframeref no)
 			(mode 1)
-			(useauxorigin no)
+			(useauxorigin yes)
 			(hpglpennumber 1)
 			(hpglpenspeed 20)
@@
 			(pdf_back_fp_property_popups yes)
 			(pdf_metadata yes)
-			(pdf_single_document yes)
+			(pdf_single_document no)
 			(dxfpolygonmode yes)
 			(dxfimperialunits yes)
@@
 			(psnegative no)
 			(psa4output no)
-			(plot_black_and_white no)
-			(sketchpadsonfab no)
-			(plotpadnumbers no)
+			(plot_black_and_white yes)
+			(sketchpadsonfab yes)
+			(plotpadnumbers yes)
 			(hidednponfab no)
 			(sketchdnponfab yes)
 			(crossoutdnponfab yes)
-			(subtractmaskfromsilk no)
-			(outputformat 4)
+			(subtractmaskfromsilk yes)
+			(outputformat 1)
 			(mirror no)
-			(drillshape 2)
+			(drillshape 0)
 			(scaleselection 1)
-			(outputdirectory "")
+			(outputdirectory "manufacturing/GERBER/")
 		)
 	)
@@
 	)
 	(segment
+		(start 210.867677 77)
+		(end 209.4 77)
+		(width 0.2)
+		(layer "F.Cu")
+		(net 1)
+	)
+	(segment
+		(start 216.042677 133.4875)
+		(end 216.042677 131.957323)
+		(width 0.2)
+		(layer "F.Cu")
+		(net 1)
+	)
+	(segment
+		(start 216.042677 131.957323)
+		(end 216.1 131.9)
+		(width 0.2)
+		(layer "F.Cu")
+		(net 1)
+	)
+	(segment
+		(start 174 66.8)
+		(end 175.6 66.8)
+		(width 0.2)
+		(layer "F.Cu")
+		(net 1)
+	)
+	(segment
+		(start 166.15 137.25)
+		(end 166.2 137.3)
+		(width 0.2)
+		(layer "F.Cu")
+		(net 1)
+	)
+	(segment
+		(start 166.15 135.9)
+		(end 166.15 137.25)
+		(width 0.2)
+		(layer "F.Cu")
+		(net 1)
+	)
+	(via
+		(at 175.6 66.8)
+		(size 0.6)
+		(drill 0.3)
+		(layers "F.Cu" "B.Cu")
+		(net 1)
+	)
+	(via
+		(at 209.4 77)
+		(size 0.6)
+		(drill 0.3)
+		(layers "F.Cu" "B.Cu")
+		(net 1)
+	)
+	(via
+		(at 216.1 131.9)
+		(size 0.6)
+		(drill 0.3)
+		(layers "F.Cu" "B.Cu")
+		(net 1)
+	)
+	(via
+		(at 166.2 137.3)
+		(size 0.6)
+		(drill 0.3)
+		(layers "F.Cu" "B.Cu")
+		(net 1)
+	)
+	(segment
+		(start 166.2 137.3)
+		(end 166.6 137.7)
+		(width 0.2)
+		(layer "B.Cu")
+		(net 1)
+	)
+	(segment
+		(start 216.1 131.9)
+		(end 216.1 131.1)
+		(width 0.2)
+		(layer "B.Cu")
+		(net 1)
+	)
+	(segment
+		(start 209.4 77)
+		(end 208.4 77)
+		(width 0.2)
+		(layer "B.Cu")
+		(net 1)
+	)
+	(segment
+		(start 175.6 66.8)
+		(end 176.4 66.8)
+		(width 0.2)
+		(layer "B.Cu")
+		(net 1)
+	)
+	(segment
